Commit message: updated anscer_navigation and anscer_description

File: anscer_description/urdf/anscer_description.xacro (robot description, xacro)
@@ -18,5 +18,4 @@
     <xacro:box_inertia m="${base_link_mass}" w="${base_len}" h="${base_height}" d="${base_width}" xyz="${base_link_offset} 0.0 ${base_wheel_gap_z}" rpy="0.0 0.0 0.0" />
     <visual>
-      <material name="red" />
       <origin xyz="0 0.0 0" rpy="0.0 0.0 0.0" />
       <geometry>

File: anscer_description/urdf/anscer_description_gazebo.xacro (robot description, xacro)
@@ -93,9 +93,4 @@
     </sensor>
   </gazebo>
-  <!-- Main body -->
-  <gazebo reference="base_link">
-    <material>Gazebo/Blue</material>
-    <turnGravityOff>false</turnGravityOff>
-  </gazebo>
   <!-- For the differential drive wheels -->
   <xacro:macro name="wheel_properties" params="prefix">

File: anscer_description/urdf/anscer_description_materials.xacro (robot description, xacro)
@@ -26,9 +26,4 @@
         <color rgba="0.0 0 0 1.0"/>
     </material>
-    <!-- Materials for Gazebo -->
-    <!-- Material for the base link -->
-    <gazebo reference="base_link">
-        <material>Gazebo/Blue</material>
-    </gazebo>
     <!-- Material for differential drive wheels -->
     <xacro:macro name="wheel_material" params="prefix">
